File: USBtoMIDI.sch (KiCad schematic (older format))
At the start: 70 parts, among them J1 Conn_01x03, J2 Conn_01x03, J3 Conn_01x03, J7 Conn_02x04_Odd_Even, J8 Conn_01x05, J9 Conn_01x09, Q1 2N2219, Q2 2N2219, Q3 2N2219, Q4 2N2219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

Commit message: changed usb type
Parts:
- USB1: footprint Connectors:USB_B -> Connectors:USB_A_Vertical; symbol Connector:USB_B -> Connector:USB_A
Changed lines of the file:
@@
 $EndComp
 $Comp
-L Connector:USB_B USB1
+L Connector:USB_A USB1
 U 1 1 6002CF10
 P 13450 2550
 F 0 "USB1" H 13507 3017 50  0000 C CNN
 F 1 "USB_B_Full" H 13507 2926 50  0000 C CNN
-F 2 "Connectors:USB_B" H 13600 2500 50  0001 C CNN
+F 2 "Connectors:USB_A_Vertical" H 13600 2500 50  0001 C CNN
 F 3 "~" H 13600 2500 50  0001 C CNN
 	1    13450 2550

Commit message: update config ports
Connections:
- net +5V: no longer J7.1 (Pin_1), J7.2 (Pin_2)
- net GND: no longer J7.7 (Pin_7), J7.8 (Pin_8)
- net MIDI_IN: now also J7.1 (Pin_1), J7.5 (Pin_5); no longer J7.3 (Pin_3)
- net MIDI_OUT: now also J7.7 (Pin_7); no longer J7.5 (Pin_5)
- net TTL_RXD: now also J7.2 (Pin_2); no longer J7.4 (Pin_4)
- net TTL_TXD: now also J7.8 (Pin_8); no longer J7.6 (Pin_6)
Other:
- note added: "1-2 Send MIDI to uC\n5-7 Loop MIDI to Outputs\n7-8 Send MIDI from uC"
Changed lines of the file:
@@
 	1    0    0    -1
 $EndComp
-Text GLabel 8100 5850 0    50   Input ~ 0
+Text GLabel 8100 5950 0    50   Input ~ 0
 MIDI_IN
-Text GLabel 8100 5950 0    50   Input ~ 0
+Text GLabel 8100 6050 0    50   Input ~ 0
 MIDI_OUT
-$Comp
-L power:GND #PWR0146
-U 1 1 601A1DE5
-P 8100 6050
-F 0 "#PWR0146" H 8100 5800 50  0001 C CNN
-F 1 "GND" V 8100 5850 50  0000 C CNN
-F 2 "" H 8100 6050 50  0001 C CNN
-F 3 "" H 8100 6050 50  0001 C CNN
-	1    8100 6050
-	0    1    1    0
-$EndComp
-$Comp
-L power:+5V #PWR0147
-U 1 1 601A27C1
-P 8100 5750
-F 0 "#PWR0147" H 8100 5600 50  0001 C CNN
-F 1 "+5V" V 8100 5900 50  0000 L CNN
-F 2 "" H 8100 5750 50  0001 C CNN
-F 3 "" H 8100 5750 50  0001 C CNN
-	1    8100 5750
-	0    -1   -1   0
-$EndComp
 $Comp
 L power:GND #PWR0148
@@
 	1    8300 5850
 	1    0    0    -1
-$EndComp
-Text GLabel 8600 5850 2    50   Input ~ 0
-TTL_RXD
-Text GLabel 8600 5950 2    50   Input ~ 0
-TTL_TXD
-$Comp
-L power:+5V #PWR0149
-U 1 1 601B6FFF
-P 8600 5750
-F 0 "#PWR0149" H 8600 5600 50  0001 C CNN
-F 1 "+5V" V 8600 5900 50  0000 L CNN
-F 2 "" H 8600 5750 50  0001 C CNN
-F 3 "" H 8600 5750 50  0001 C CNN
-	1    8600 5750
-	0    1    1    0
-$EndComp
-$Comp
-L power:GND #PWR0150
-U 1 1 601B7A49
-P 8600 6050
-F 0 "#PWR0150" H 8600 5800 50  0001 C CNN
-F 1 "GND" V 8600 5850 50  0000 C CNN
-F 2 "" H 8600 6050 50  0001 C CNN
-F 3 "" H 8600 6050 50  0001 C CNN
-	1    8600 6050
-	0    -1   -1   0
 $EndComp
 Text GLabel 11350 2650 2    50   Input ~ 0
@@
 Wire Wire Line
 	7800 7500 7900 7500
+Text GLabel 8100 5750 0    50   Input ~ 0
+MIDI_IN
+Text GLabel 8600 5750 2    50   Input ~ 0
+TTL_RXD
+Text GLabel 8600 6050 2    50   Input ~ 0
+TTL_TXD
+Text Notes 7900 6400 0    50   ~ 0
+1-2 Send MIDI to uC\n5-7 Loop MIDI to Outputs\n7-8 Send MIDI from uC
 $EndSCHEMATC

Commit message: update logic
Parts:
- added unit 6 of U4
- added unit 5 of U4
- U4, U5: value 74HC14 -> 74AS14
- U5: renamed from U4; value 74HC14 -> 74AS14
- U7: value 4081 -> 74HC08
Connections:
- net GND: now also Q3.1 (E), U4.3, U4.4
- net MIDI_IN: now also U4.2, U4.5; no longer R24.1, U4.4
- net at U7.3: now also U4.13; no longer U4.5
- net at R22.1: now also U4.10; no longer U4.8
- net at U5.10: now also R21.1; no longer R15.1
- net at U5.13: now also U7.11; no longer U7.4
- net at U5.4: now also R15.1; no longer R18.1
- net at U5.8: now also R18.1; no longer R21.1
- net at U5.1: now also U7.4; no longer U7.10
- net at U5.5: now also U7.10; no longer U7.11
- new net: U4.11, U4.12
- new net: R24.1, U4.8
Other:
- moved on the sheet: R10, R11, R12, R25, R26, R27, R9, U4B, U4C, U4D, U4G, U5A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

Commit message: updates
Parts:
- D1: footprint Diodes_SMD:D_1206 -> Diodes_SMD:D_SOD-323
- U6: footprint Housings_DIP:SMDIP-8_W7.62mm -> Housings_DIP:DIP-8_W7.62mm
Connections:
- net at U5.10: now also R18.1; no longer R21.1
- net at U5.13: now also U7.10; no longer U7.11
- net at U5.8: now also R21.1; no longer R18.1
- net at U5.5: now also U7.11; no longer U7.10
Other:
- moved on the sheet: J7, R25, R26, R27, R28, SW1, U5C, U5D, U5E, U5F, USB1, USB2

Commit message: updates
Parts:
- R8: value 100R -> 220R
Connections:
- net +5V: now also J7.3 (Pin_3)
- net GND: now also J7.4 (Pin_4), J7.6 (Pin_6)
Changed lines of the file:
@@
 P 2950 1150
 F 0 "R8" V 2743 1150 50  0000 C CNN
-F 1 "100R" V 2834 1150 50  0000 C CNN
+F 1 "220R" V 2834 1150 50  0000 C CNN
 F 2 "Resistors_SMD:R_0805_HandSoldering" V 2880 1150 50  0001 C CNN
 F 3 "~" H 2950 1150 50  0001 C CNN
@@
 Wire Wire Line
 	2650 2550 3000 2550
+$Comp
+L power:GND #PWR?
+U 1 1 6009D47E
+P 9100 5900
+F 0 "#PWR?" H 9100 5650 50  0001 C CNN
+F 1 "GND" V 9100 5700 50  0000 C CNN
+F 2 "" H 9100 5900 50  0001 C CNN
+F 3 "" H 9100 5900 50  0001 C CNN
+	1    9100 5900
+	0    -1   -1   0
+$EndComp
+$Comp
+L power:+5V #PWR?
+U 1 1 6009D8BB
+P 8600 5900
+F 0 "#PWR?" H 8600 5750 50  0001 C CNN
+F 1 "+5V" V 8600 6100 50  0000 C CNN
+F 2 "" H 8600 5900 50  0001 C CNN
+F 3 "" H 8600 5900 50  0001 C CNN
+	1    8600 5900
+	0    -1   -1   0
+$EndComp
+$Comp
+L power:GND #PWR?
+U 1 1 600B28DF
+P 9100 6000
+F 0 "#PWR?" H 9100 5750 50  0001 C CNN
+F 1 "GND" V 9100 5800 50  0000 C CNN
+F 2 "" H 9100 6000 50  0001 C CNN
+F 3 "" H 9100 6000 50  0001 C CNN
+	1    9100 6000
+	0    -1   -1   0
+$EndComp
 $EndSCHEMATC
